File: kicad/pccs.kicad_sch (KiCad schematic)
At the start: 230 parts, among them J1 Power, J2 Analog In, J3 Analog In, J4 Digital, J5 Communication, J6 PWM, J7 PWM, K1 Relay_SPDT, K2 Relay_SPDT, K3 Relay_SPDT, K4 Relay_SPDT, Q1 IRLB8721PBF, Q10 IRLB8721PBF, Q11 IRLB8721PBF, Q12 IRLB8721PBF, Q13 IRLB8721PBF, Q14 IRLB8721PBF, Q15 IRLB8721PBF, Q16 IRLZ44N, Q17 IRLZ44N, Q18 IRLZ44N, Q19 IRLZ44N, Q2 IRLB8721PBF, Q3 IRLB8721PBF, Q4 IRLB8721PBF, Q5 IRLB8721PBF, Q6 IRLB8721PBF, Q7 IRLB8721PBF, Q8 IRLB8721PBF, Q9 IRLB8721PBF, U1 PC817, U2 PC817, U3 PC817, U4 PC817, U5 TPS568215RNN

Commit message: Update KiCad footprints
Parts:
- C17, C19, C21, C23: LCSC Part # C165558 -> C44587
- C28: footprint Capacitor_THT:CP_Radial_D8.0mm_P3.50mm -> Capacitor_SMD:CP_Elec_8x10
- D10, D15, D19, D5: value MBR1045 -> (none); footprint Package_TO_SOT_THT:TO-220-2_Vertical -> Diode_SMD:D_PowerDI-5; LCSC Part # C260253 -> C2759901
- D28: value 1N5822 -> (none); footprint Package_TO_SOT_THT:TO-220-2_Vertical -> Diode_SMD:D_PowerDI-5; LCSC Part # C2476 -> C2759901
- D29: footprint Diode_SMD:Nexperia_DSN1608-2_1.6x0.8mm -> Diode_SMD:D_SMB; LCSC Part # C118306 -> C571369
- L1: value 15uH -> 3.3uH; footprint Inductor_SMD:L_10.4x10.4_H4.8 -> Inductor_SMD:L_SXN_SMDRI127; LCSC Part # C16113 -> C24550
- U1, U2, U3, U4: footprint Package_DIP:DIP-4_W7.62mm -> Package_DIP:DIP-4_W10.16mm
Other:
- note removed: "L1 needs to be 3A saturation"
- note removed: "L2 needs to be 10A saturation"

Commit message: Standardized screw connectors manufacturer
Parts:
- J1, J2, J3, J5, J6: LCSC Part # (none) -> C27438; now in the parts list
- J4: LCSC Part # (none) -> C132131; now in the parts list
- J7: LCSC Part # (none) -> C35445; now in the parts list
- PI1: LCSC Part # (none) -> C132132; now in the parts list
- U1, U2, U3, U4: footprint Package_DIP:DIP-4_W10.16mm -> Package_DIP:DIP-4_W7.62mm; LCSC Part # C41807 -> C5353
- i1: LCSC Part # C5482573 -> C508906
- i2, i3: LCSC Part # C480509 -> C8412
- i4, i5, i6, i8: LCSC Part # C480503 -> C8445
- pwm1, pwm2, pwm3: LCSC Part # C3019624 -> C29173
- pwm4: LCSC Part # C480562 -> C15084
- re1, re2, re3, re4: LCSC Part # C457197 -> C8423
Changed lines of the file:
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@@
 		(body_style 1)
 		(exclude_from_sim no)
-		(in_bom no)
+		(in_bom yes)
 		(on_board yes)
 		(in_pos_files yes)
@@
 			)
 		)
-		(property "LCSC Part #" ""
+		(property "LCSC Part #" "C35445"
 			(at 208.28 198.12 90)
 			(hide yes)
@@
 		(body_style 1)
 		(exclude_from_sim no)
-		(in_bom no)
+		(in_bom yes)
 		(on_board yes)
 		(in_pos_files yes)
@@
 			)
 		)
-		(property "LCSC Part #" ""
+		(property "LCSC Part #" "C27438"
 			(at 162.56 198.12 90)
 			(hide yes)
@@
 		(body_style 1)
 		(exclude_from_sim no)
-		(in_bom no)
+		(in_bom yes)
 		(on_board yes)
 		(in_pos_files yes)
@@
 			)
 		)
-		(property "LCSC Part #" ""
+		(property "LCSC Part #" "C27438"
 			(at 182.88 198.12 90)
 			(hide yes)
@@
 			)
 		)
-		(property "Footprint" "Package_DIP:DIP-4_W10.16mm"
+		(property "Footprint" "Package_DIP:DIP-4_W7.62mm"
 			(at 471.17 262.89 0)
 			(hide yes)
@@
 			)
 		)
-		(property "LCSC Part #" "C41807"
+		(property "LCSC Part #" "C5353"
 			(at 466.09 267.97 90)
 			(hide yes)
@@
 			)
 		)
-		(property "LCSC Part #" "C457197"
+		(property "LCSC Part #" "C8423"
 			(at 551.18 342.9 0)
 			(hide yes)
@@
 			)
 		)
-		(property "LCSC Part #" "C480503"
+		(property "LCSC Part #" "C8445"
 			(at 43.18 267.97 0)
 			(hide yes)
@@
 			)
 		)
-		(property "Footprint" "Package_DIP:DIP-4_W10.16mm"
+		(property "Footprint" "Package_DIP:DIP-4_W7.62mm"
 			(at 471.17 321.31 0)
 			(hide yes)
@@
 			)
 		)
-		(property "LCSC Part #" "C41807"
+		(property "LCSC Part #" "C5353"
 			(at 466.09 326.39 90)
 			(hide yes)
@@
 		(body_style 1)
 		(exclude_from_sim no)
-		(in_bom no)
+		(in_bom yes)
 		(on_board yes)
 		(in_pos_files yes)
@@
 			)
 		)
-		(property "LCSC Part #" ""
+		(property "LCSC Part #" "C27438"
 			(at 166.37 254 90)
 			(hide yes)
@@
 			)
 		)
-		(property "LCSC Part #" "C480503"
+		(property "LCSC Part #" "C8445"
 			(at 41.91 364.49 0)
 			(hide yes)
@@
 		(body_style 1)
 		(exclude_from_sim no)
-		(in_bom no)
+		(in_bom yes)
 		(on_board yes)
 		(in_pos_files yes)
@@
 			)
 		)
-		(property "LCSC Part #" ""
+		(property "LCSC Part #" "C27438"
 			(at 191.77 254 90)
 			(hide yes)
@@
 		(body_style 1)
 		(exclude_from_sim no)
-		(in_bom no)
+		(in_bom yes)
 		(on_board yes)
 		(in_pos_files yes)
@@
 			)
 		)
-		(property "LCSC Part #" ""
+		(property "LCSC Part #" "C132131"
 			(at 142.24 227.33 0)
 			(hide yes)
@@
 			)
 		)
-		(property "LCSC Part #" "C480509"
+		(property "LCSC Part #" "C8412"
 			(at 41.91 161.29 0)
 			(hide yes)
@@
 			)
 		)
-		(property "LCSC Part #" "C480509"
+		(property "LCSC Part #" "C8412"
 			(at 41.91 127 0)
 			(hide yes)
@@
 			)
 		)
-		(property "LCSC Part #" "C457197"
+		(property "LCSC Part #" "C8423"
 			(at 411.48 284.48 0)
 			(hide yes)
@@
 			)
 		)
-		(property "LCSC Part #" "C3019624"
+		(property "LCSC Part #" "C29173"
 			(at 546.1 50.8 0)
 			(hide yes)
@@
 			)
 		)
-		(property "LCSC Part #" "C480503"
+		(property "LCSC Part #" "C8445"
 			(at 43.18 217.17 0)
 			(hide yes)
@@
 			)
 		)
-		(property "LCSC Part #" "C457197"
+		(property "LCSC Part #" "C8423"
 			(at 411.48 342.9 0)
 			(hide yes)
@@
 			)
 		)
-		(property "LCSC Part #" "C5482573"
+		(property "LCSC Part #" "C508906"
 			(at 41.91 54.61 0)
 			(hide yes)
@@
 		(body_style 1)
 		(exclude_from_sim no)
-		(in_bom no)
+		(in_bom yes)
 		(on_board yes)
 		(in_pos_files yes)
@@
 			)
 		)
-		(property "LCSC Part #" ""
+		(property "LCSC Part #" "C132132"
 			(at 217.17 67.31 0)
 			(hide yes)
@@
 			)
 		)
-		(property "Footprint" "Package_DIP:DIP-4_W10.16mm"
+		(property "Footprint" "Package_DIP:DIP-4_W7.62mm"
 			(at 331.47 321.31 0)
 			(hide yes)
@@
 			)
 		)
-		(property "LCSC Part #" "C41807"
+		(property "LCSC Part #" "C5353"
 			(at 326.39 326.39 90)
 			(hide yes)
@@
 			)
 		)
-		(property "LCSC Part #" "C480503"
+		(property "LCSC Part #" "C8445"
 			(at 43.18 242.57 0)
 			(hide yes)
@@
 			)
 		)
-		(property "Footprint" "Package_DIP:DIP-4_W10.16mm"
+		(property "Footprint" "Package_DIP:DIP-4_W7.62mm"
 			(at 331.47 262.89 0)
 			(hide yes)
@@
 			)
 		)
-		(property "LCSC Part #" "C41807"
+		(property "LCSC Part #" "C5353"
 			(at 326.39 267.97 90)
 			(hide yes)
@@
 			)
 		)
-		(property "LCSC Part #" "C457197"
+		(property "LCSC Part #" "C8423"
 			(at 551.18 284.48 0)
 			(hide yes)
@@
 			)
 		)
-		(property "LCSC Part #" "C3019624"
+		(property "LCSC Part #" "C29173"
 			(at 546.1 104.14 0)
 			(hide yes)
@@
 			)
 		)
-		(property "LCSC Part #" "C480562"
+		(property "LCSC Part #" "C15084"
 			(at 546.1 208.28 0)
 			(hide yes)
@@
 			)
 		)
-		(property "LCSC Part #" "C3019624"
+		(property "LCSC Part #" "C29173"
 			(at 546.1 157.48 0)
 			(hide yes)
@@
 		(body_style 1)
 		(exclude_from_sim no)
-		(in_bom no)
+		(in_bom yes)
 		(on_board yes)
 		(in_pos_files yes)
@@
 			)
 		)
-		(property "LCSC Part #" ""
+		(property "LCSC Part #" "C27438"
 			(at 217.17 254 90)
 			(hide yes)
